Commit message: Added mobile robot model, fixed DoF of control parameters.

File: src/model/robot.urdf (robot description, URDF)
Before this commit: robot panda, 29 links, 28 joints
Links:
- added link omni_base_root_link
- added link pivot, mass 0.01
- added link x_slider, mass 0.01
- added link y_slider, mass 0.01
- link axle_link: geometry visual mesh filename=ridgeback/meshes/axle.obj
- link base_link: geometry collision box size=0.20 0.90 0.55; collision box size=0.95 0.90 0.5
- link chassis_link: geometry visual mesh filename=ridgeback/meshes/body.obj
- link front_cover_link: geometry visual mesh filename=ridgeback/meshes/end-cover.obj
- link front_lights_link: geometry visual mesh filename=ridgeback/meshes/lights.obj
- link left_side_cover_link: geometry visual mesh filename=ridgeback/meshes/side-cover.obj
- link panda_hand: geometry collision box size=0.035 0.19 0.065; visual mesh filename=panda/meshes/visual/hand.dae
- link panda_leftfinger: geometry collision box size=0.0222 0.007 0.025; collision box size=0.0222 0.0145 0.018
- link panda_link0: geometry collision mesh filename=panda/meshes/collision/link0.obj; visual mesh filename=panda/meshes/visual/link0.dae
- link panda_link1: geometry collision mesh filename=panda/meshes/collision/link1.obj; visual mesh filename=panda/meshes/visual/link1.dae
- link panda_link2: geometry collision mesh filename=panda/meshes/collision/link2.obj; visual mesh filename=panda/meshes/visual/link2.dae
- link panda_link3: geometry collision mesh filename=panda/meshes/collision/link3.obj; visual mesh filename=panda/meshes/visual/link3.dae
- link panda_link4: geometry collision mesh filename=panda/meshes/collision/link4.obj; visual mesh filename=panda/meshes/visual/link4.dae
- link panda_link5: geometry collision mesh filename=panda/meshes/collision/link5.obj; visual mesh filename=panda/meshes/visual/link5.dae
- link panda_link6: geometry collision mesh filename=panda/meshes/collision/link6.obj; visual mesh filename=panda/meshes/visual/link6.dae
- link panda_link7: geometry collision mesh filename=panda/meshes/collision/link7.obj; visual mesh filename=panda/meshes/visual/link7.dae
- link panda_rightfinger: geometry collision box size=0.0222 0.007 0.025; collision box size=0.0222 0.0145 0.018
- link rear_cover_link: geometry visual mesh filename=ridgeback/meshes/end-cover.obj
- link rear_lights_link: geometry visual mesh filename=ridgeback/meshes/lights.obj
- link ridgeback_sensor_mount_link: geometry 
- link right_side_cover_link: geometry visual mesh filename=ridgeback/meshes/side-cover.obj
- link top_link: geometry visual mesh filename=ridgeback/meshes/top.obj
Joints:
- added joint omni_base_flange: type fixed, parent pivot, child base_link
- added joint pivot_joint: type revolute, parent y_slider, child pivot, origin xyz=0.0 0.0 0.0 rpy=0 0 0, axis 0 0 1, limit lower=-10.0 upper=10.0 effort=1000.0 velocity=1.0
- added joint x_base_joint: type prismatic, parent omni_base_root_link, child x_slider, origin xyz=0.0 0.0 0.0 rpy=0 0 0, axis 1 0 0, limit lower=-10 upper=10 effort=1000.0 velocity=1.0
- added joint y_base_joint: type prismatic, parent x_slider, child y_slider, origin xyz=0.0 0.0 0.0 rpy=0 0 0, axis 0 1 0, limit lower=-10 upper=10 effort=1000.0 velocity=1.0
- joint arm_mount_joint: origin xyz=0.30 0.0 0.445 rpy=0 0 0 -> xyz=0.295 0.005 0.445 rpy=0 0 0
- joint panda_grasp_joint: origin xyz=0 0 0.1 rpy=0 0 0 -> xyz=0 0 0.095 rpy=0 0 0
- joint panda_joint1: limit lower=-20 upper=20 effort=87 velocity=2.1750 -> lower=-2.8973 upper=2.8973 effort=87 velocity=2.1750
- joint panda_joint2: limit lower=-20 upper=20 effort=87 velocity=2.1750 -> lower=-1.7628 upper=1.7628 effort=87 velocity=2.1750
- joint panda_joint3: limit lower=-20 upper=20 effort=87 velocity=2.1750 -> lower=-2.8973 upper=2.8973 effort=87 velocity=2.1750
- joint panda_joint4: limit lower=-20 upper=20 effort=87 velocity=2.1750 -> lower=-3.0718 upper=0.0698 effort=87 velocity=2.1750
- joint panda_joint5: limit lower=-20 upper=20 effort=12 velocity=2.6100 -> lower=-2.8973 upper=2.8973 effort=12 velocity=2.6100
- joint panda_joint6: limit lower=-20 upper=20 effort=12 velocity=2.6100 -> lower=-0.0175 upper=3.7525 effort=12 velocity=2.6100
- joint panda_joint7: limit lower=-20 upper=20 effort=12 velocity=2.6100 -> lower=-2.8973 upper=2.8973 effort=12 velocity=2.6100
- joint world_joint: child base_link -> omni_base_root_link; origin xyz=0.004 1.087 0.000 rpy=0.000 0.000 -1.500 -> (none)
