Commit message: Forecast logging, moved objective config, fixes. - Added logging the forecast dynamics. - Moved configuration of the objective function to   the frankaridgeback actor. - Added FrankaRidgeback namespace to objective   functions. - Fixed self collision link names using constants. - Removed cyan circle visual from model. - Updated assisted manipulation objective function.   - Implemented self collision with intersecting     spheres.   - Implemented basic trajectory following.

File: src/frankaridgeback/model/ridgeback.xacro (robot description, xacro)
@@ -27,5 +27,5 @@
             <inertia ixx="0.048966669" ixy="0" ixz="0" iyy="0.046466667" iyz="0" izz="0.0041666669"/>
         </inertial>
-        <visual>
+        <!-- <visual>
             <origin xyz="0 0 0" rpy="0 0 0" />
             <geometry>
@@ -35,5 +35,5 @@
                <color rgba="0 1.0 1.0 0.3"/>
             </material>
-        </visual>
+        </visual> -->
        <collision>
            <origin rpy="0 0 0" xyz="0 0 0.25"/>

File: src/frankaridgeback/model/robot.urdf (robot description, URDF)
Before this commit: robot panda, 33 links, 32 joints
Links:
- link base_link: geometry collision box size=0.20 0.90 0.55; collision box size=0.95 0.90 0.5
